Commit message: Final refactor changes to ur5_apla

File: src/ur5_apla/urdf/ur5_apla.xacro (robot description, xacro)
@@ -1,358 +1,30 @@
-<?xml version="1.0" ?>
-<robot name="ur5_apla">
-    <!--
-    Base UR robot series xacro macro.
-    NOTE: this is NOT a URDF. It cannot directly be loaded by consumers
-    expecting a flattened '.urdf' file. See the top-level '.xacro' for that
-    (but note: that .xacro must still be processed by the xacro command).
-    For use in '.launch' files: use one of the 'load_urX.launch' convenience
-    launch files.
-    This file models the base kinematic chain of a UR robot, which then gets
-    parameterised by various configuration files to convert it into a UR3(e),
-    UR5(e), UR10(e), UR16e, UR20 or UR30.
-    NOTE: the default kinematic parameters (ie: link lengths, frame locations,
-    offets, etc) do not correspond to any particular robot. They are defaults
-    only. There WILL be non-zero offsets between the Forward Kinematics results
-    in TF (ie: robot_state_publisher) and the values reported by the Teach
-    Pendant.
-    For accurate (and robot-specific) transforms, the 'kinematics_parameters_file'
-    parameter MUST point to a .yaml file containing the appropriate values for
-    the targetted robot.
-    If using the UniversalRobots/Universal_Robots_ROS_Driver, follow the steps
-    described in the readme of that repository to extract the kinematic
-    calibration from the controller and generate the required .yaml file.
-    Main author of the migration to yaml configs: Ludovic Delval.
-    Contributors to previous versions (in no particular order):
-     - Felix Messmer
-     - Kelsey Hawkins
-     - Wim Meeussen
-     - Shaun Edwards
-     - Nadia Hammoudeh Garcia
-     - Dave Hershberger
-     - G. vd. Hoorn
-     - Philip Long
-     - Dave Coleman
-     - Miguel Prada
-     - Mathias Luedtke
-     - Marcel Schnirring
-     - Felix von Drigalski
-     - Felix Exner
-     - Jimmy Da Silva
-     - Ajit Krisshna N L
-     - Muhammad Asif Rana
-  -->
-    <transmission name="shoulder_pan_trans">
-        <type>transmission_interface/SimpleTransmission</type>
-        <joint name="shoulder_pan_joint">
-            <hardwareInterface>hardware_interface/PositionJointInterface</hardwareInterface>
-        </joint>
-        <actuator name="shoulder_pan_motor">
-            <mechanicalReduction>1</mechanicalReduction>
-            <hardwareInterface>hardware_interface/EffortJointInterface</hardwareInterface>
-        </actuator>
-    </transmission>
-    <transmission name="shoulder_lift_trans">
-        <type>transmission_interface/SimpleTransmission</type>
-        <joint name="shoulder_lift_joint">
-            <hardwareInterface>hardware_interface/PositionJointInterface</hardwareInterface>
-        </joint>
-        <actuator name="shoulder_lift_motor">
-            <mechanicalReduction>1</mechanicalReduction>
-            <hardwareInterface>hardware_interface/EffortJointInterface</hardwareInterface>
-        </actuator>
-    </transmission>
-    <transmission name="elbow_trans">
-        <type>transmission_interface/SimpleTransmission</type>
-        <joint name="elbow_joint">
-            <hardwareInterface>hardware_interface/PositionJointInterface</hardwareInterface>
-        </joint>
-        <actuator name="elbow_motor">
-            <mechanicalReduction>1</mechanicalReduction>
-            <hardwareInterface>hardware_interface/EffortJointInterface</hardwareInterface>
-        </actuator>
-    </transmission>
-    <transmission name="wrist_1_trans">
-        <type>transmission_interface/SimpleTransmission</type>
-        <joint name="wrist_1_joint">
-            <hardwareInterface>hardware_interface/PositionJointInterface</hardwareInterface>
-        </joint>
-        <actuator name="wrist_1_motor">
-            <mechanicalReduction>1</mechanicalReduction>
-            <hardwareInterface>hardware_interface/EffortJointInterface</hardwareInterface>
-        </actuator>
-    </transmission>
-    <transmission name="wrist_2_trans">
-        <type>transmission_interface/SimpleTransmission</type>
-        <joint name="wrist_2_joint">
-            <hardwareInterface>hardware_interface/PositionJointInterface</hardwareInterface>
-        </joint>
-        <actuator name="wrist_2_motor">
-            <mechanicalReduction>1</mechanicalReduction>
-            <hardwareInterface>hardware_interface/EffortJointInterface</hardwareInterface>
-        </actuator>
-    </transmission>
-    <transmission name="wrist_3_trans">
-        <type>transmission_interface/SimpleTransmission</type>
-        <joint name="wrist_3_joint">
-            <hardwareInterface>hardware_interface/PositionJointInterface</hardwareInterface>
-        </joint>
-        <actuator name="wrist_3_motor">
-            <mechanicalReduction>1</mechanicalReduction>
-            <hardwareInterface>hardware_interface/EffortJointInterface</hardwareInterface>
-        </actuator>
-    </transmission>
-    <!-- links: main serial chain -->
-    <link name="base_link" />
-    <link name="base_link_inertia">
-        <visual>
-            <origin rpy="0 0 3.141592653589793" xyz="0 0 0" />
-            <geometry>
-                <mesh filename="package://ur5_apla/meshes/ur5/visual/base.dae" />
-            </geometry>
-            <material name="LightGrey">
-                <color rgba="0.7 0.7 0.7 1.0" />
-            </material>
-        </visual>
-        <collision>
-            <origin rpy="0 0 3.141592653589793" xyz="0 0 0" />
-            <geometry>
-                <mesh filename="package://ur5_apla/meshes/ur5/collision/base.stl" />
-            </geometry>
-        </collision>
-        <inertial>
-            <mass value="4.0" />
-            <origin rpy="0 0 0" xyz="0 0 0" />
-            <inertia ixx="0.00443333156" ixy="0.0" ixz="0.0" iyy="0.00443333156" iyz="0.0" izz="0.0072" />
-        </inertial>
-    </link>
-    <!--Fix the robot to the world, added by Tim -->
-<!--<link name="world"/>
-    <joint name="fixed" type="fixed">
-        <parent link="world"/>
-        <child link="base_link"/>
-    </joint>-->
-    <link name="shoulder_link">
-        <visual>
-            <origin rpy="0 0 3.141592653589793" xyz="0 0 0" />
-            <geometry>
-                <mesh filename="package://ur5_apla/meshes/ur5/visual/shoulder.dae" />
-            </geometry>
-            <material name="LightGrey">
-                <color rgba="0.7 0.7 0.7 1.0" />
-            </material>
-        </visual>
-        <collision>
-            <origin rpy="0 0 3.141592653589793" xyz="0 0 0" />
-            <geometry>
-                <mesh filename="package://ur5_apla/meshes/ur5/collision/shoulder.stl" />
-            </geometry>
-        </collision>
-        <inertial>
-            <mass value="3.7" />
-            <origin rpy="0 0 0" xyz="0 0 0" />
-            <inertia ixx="0.014972352344389999" ixy="0.0" ixz="0.0" iyy="0.014972352344389999" iyz="0.0" izz="0.01040625" />
-        </inertial>
-    </link>
-    <link name="upper_arm_link">
-        <visual>
-            <origin rpy="1.5707963267948966 0 -1.5707963267948966" xyz="0 0 0.13585" />
-            <geometry>
-                <mesh filename="package://ur5_apla/meshes/ur5/visual/upperarm.dae" />
-            </geometry>
-            <material name="LightGrey">
-                <color rgba="0.7 0.7 0.7 1.0" />
-            </material>
-        </visual>
-        <collision>
-            <origin rpy="1.5707963267948966 0 -1.5707963267948966" xyz="0 0 0.13585" />
-            <geometry>
-                <mesh filename="package://ur5_apla/meshes/ur5/collision/upperarm.stl" />
-            </geometry>
-        </collision>
-        <inertial>
-            <mass value="8.393" />
-            <origin rpy="0 1.5707963267948966 0" xyz="-0.2125 0.0 0.136" />
-            <inertia ixx="0.1338857818623325" ixy="0.0" ixz="0.0" iyy="0.1338857818623325" iyz="0.0" izz="0.0151074" />
-        </inertial>
-    </link>
-    <link name="forearm_link">
-        <visual>
-            <origin rpy="1.5707963267948966 0 -1.5707963267948966" xyz="0 0 0.0165" />
-            <geometry>
-                <mesh filename="package://ur5_apla/meshes/ur5/visual/forearm.dae" />
-            </geometry>
-            <material name="LightGrey">
-                <color rgba="0.7 0.7 0.7 1.0" />
-            </material>
-        </visual>
-        <collision>
-            <origin rpy="1.5707963267948966 0 -1.5707963267948966" xyz="0 0 0.0165" />
-            <geometry>
-                <mesh filename="package://ur5_apla/meshes/ur5/collision/forearm.stl" />
-            </geometry>
-        </collision>
-        <inertial>
-            <mass value="2.275" />
-            <origin rpy="0 1.5707963267948966 0" xyz="-0.196125 0.0 0.0165" />
-            <inertia ixx="0.03121679102890359" ixy="0.0" ixz="0.0" iyy="0.03121679102890359" iyz="0.0" izz="0.004095" />
-        </inertial>
-    </link>
-    <link name="wrist_1_link">
-        <visual>
-            <!-- TODO: Move this to a parameter -->
-            <origin rpy="1.5707963267948966 0 0" xyz="0 0 -0.093" />
-            <geometry>
-                <mesh filename="package://ur5_apla/meshes/ur5/visual/wrist1.dae" />
-            </geometry>
-            <material name="LightGrey">
-                <color rgba="0.7 0.7 0.7 1.0" />
-            </material>
-        </visual>
-        <collision>
-            <origin rpy="1.5707963267948966 0 0" xyz="0 0 -0.093" />
-            <geometry>
-                <mesh filename="package://ur5_apla/meshes/ur5/collision/wrist1.stl" />
-            </geometry>
-        </collision>
-        <inertial>
-            <mass value="1.219" />
-            <origin rpy="0 0 0" xyz="0 0 0" />
-            <inertia ixx="0.0020138887777775" ixy="0.0" ixz="0.0" iyy="0.0020138887777775" iyz="0.0" izz="0.0021942" />
-        </inertial>
-    </link>
-    <link name="wrist_2_link">
-        <visual>
-            <origin rpy="0 0 0" xyz="0 0 -0.095" />
-            <geometry>
-                <mesh filename="package://ur5_apla/meshes/ur5/visual/wrist2.dae" />
-            </geometry>
-            <material name="LightGrey">
-                <color rgba="0.7 0.7 0.7 1.0" />
-            </material>
-        </visual>
-        <collision>
-            <origin rpy="0 0 0" xyz="0 0 -0.095" />
-            <geometry>
-                <mesh filename="package://ur5_apla/meshes/ur5/collision/wrist2.stl" />
-            </geometry>
-        </collision>
-        <inertial>
-            <mass value="1.219" />
-            <origin rpy="0 0 0" xyz="0 0 0" />
-            <inertia ixx="0.0018310388509175" ixy="0.0" ixz="0.0" iyy="0.0018310388509175" iyz="0.0" izz="0.0021942" />
-        </inertial>
-    </link>
-    <link name="wrist_3_link">
-        <visual>
-            <origin rpy="1.5707963267948966 0 0" xyz="0 0 -0.0818" />
-            <geometry>
-                <mesh filename="package://ur5_apla/meshes/ur5/visual/wrist3.dae" />
-            </geometry>
-            <material name="LightGrey">
-                <color rgba="0.7 0.7 0.7 1.0" />
-            </material>
-        </visual>
-        <collision>
-            <origin rpy="1.5707963267948966 0 0" xyz="0 0 -0.0818" />
-            <geometry>
-                <mesh filename="package://ur5_apla/meshes/ur5/collision/wrist3.stl" />
-            </geometry>
-        </collision>
-        <inertial>
-            <mass value="0.1879" />
-            <origin rpy="0 0 0" xyz="0.0 0.0 -0.01525" />
-            <inertia ixx="8.062472608343e-05" ixy="0.0" ixz="0.0" iyy="8.062472608343e-05" iyz="0.0" izz="0.0001321171875" />
-        </inertial>
-    </link>
-    <!-- joints: main serial chain -->
-    <joint name="base_link-base_link_inertia" type="fixed">
-        <parent link="base_link" />
-        <child link="base_link_inertia" />
-        <!-- 'base_link' is REP-103 aligned (so X+ forward), while the internal
-           frames of the robot/controller have X+ pointing backwards.
-           Use the joint between 'base_link' and 'base_link_inertia' (a dummy
-           link/frame) to introduce the necessary rotation over Z (of pi rad).
-      -->
-        <origin rpy="0 0 3.141592653589793" xyz="0 0 0" />
-    </joint>
-    <joint name="shoulder_pan_joint" type="revolute">
-        <parent link="base_link_inertia" />
-        <child link="shoulder_link" />
-        <origin rpy="0 0 0" xyz="0 0 0.089159" />
-        <axis xyz="0 0 1" />
-        <limit effort="150.0" lower="-6.283185307179586" upper="6.283185307179586" velocity="3.141592653589793" />
-        <dynamics damping="0" friction="0" />
-    </joint>
-    <joint name="shoulder_lift_joint" type="revolute">
-        <parent link="shoulder_link" />
-        <child link="upper_arm_link" />
-        <origin rpy="1.570796327 0 0" xyz="0 0 0" />
-        <axis xyz="0 0 1" />
-        <limit effort="150.0" lower="-6.283185307179586" upper="6.283185307179586" velocity="3.141592653589793" />
-        <dynamics damping="0" friction="0" />
-    </joint>
-    <joint name="elbow_joint" type="revolute">
-        <parent link="upper_arm_link" />
-        <child link="forearm_link" />
-        <origin rpy="0 0 0" xyz="-0.425 0 0" />
-        <axis xyz="0 0 1" />
-        <limit effort="150.0" lower="-3.141592653589793" upper="3.141592653589793" velocity="3.141592653589793" />
-        <dynamics damping="0" friction="0" />
-    </joint>
-    <joint name="wrist_1_joint" type="revolute">
-        <parent link="forearm_link" />
-        <child link="wrist_1_link" />
-        <origin rpy="0 0 0" xyz="-0.39225 0 0.10915" />
-        <axis xyz="0 0 1" />
-        <limit effort="28.0" lower="-6.283185307179586" upper="6.283185307179586" velocity="3.141592653589793" />
-        <dynamics damping="0" friction="0" />
-    </joint>
-    <joint name="wrist_2_joint" type="revolute">
-        <parent link="wrist_1_link" />
-        <child link="wrist_2_link" />
-        <origin rpy="1.570796327 0 0" xyz="0 -0.09465 -1.941303950897609e-11" />
-        <axis xyz="0 0 1" />
-        <limit effort="28.0" lower="-6.283185307179586" upper="6.283185307179586" velocity="3.141592653589793" />
-        <dynamics damping="0" friction="0" />
-    </joint>
-    <joint name="wrist_3_joint" type="revolute">
-        <parent link="wrist_2_link" />
-        <child link="wrist_3_link" />
-        <origin rpy="1.570796326589793 3.141592653589793 3.141592653589793" xyz="0 0.0823 -1.688001216681175e-11" />
-        <axis xyz="0 0 1" />
-        <limit effort="28.0" lower="-6.283185307179586" upper="6.283185307179586" velocity="3.141592653589793" />
-        <dynamics damping="0" friction="0" />
-    </joint>
-    <!-- ROS-Industrial 'base' frame: base_link to UR 'Base' Coordinates transform -->
-    <link name="base" />
-    <joint name="base_link-base_fixed_joint" type="fixed">
-        <!-- Note the rotation over Z of pi radians: as base_link is REP-103
-           aligned (ie: has X+ forward, Y+ left and Z+ up), this is needed
-           to correctly align 'base' with the 'Base' coordinate system of
-           the UR controller.
-      -->
-        <origin rpy="0 0 3.141592653589793" xyz="0 0 0" />
-        <parent link="base_link" />
-        <child link="base" />
-    </joint>
-    <!-- ROS-Industrial 'flange' frame: attachment point for EEF models -->
-    <link name="flange" />
-    <joint name="wrist_3-flange" type="fixed">
-        <parent link="wrist_3_link" />
-        <child link="flange" />
-        <origin rpy="0 -1.5707963267948966 -1.5707963267948966" xyz="0 0 0" />
-    </joint>
-    <!-- ROS-Industrial 'tool0' frame: all-zeros tool frame -->
-    <link name="tool0" />
-    <joint name="flange-tool0" type="fixed">
-        <!-- default toolframe: X+ left, Y+ up, Z+ front -->
-        <origin rpy="1.5707963267948966 0 1.5707963267948966" xyz="0 0 0" />
-        <parent link="flange" />
-        <child link="tool0" />
-    </joint>
-    <gazebo>
-        <plugin name="gazebo_ros_control" filename="libgazebo_ros_control.so">
-            <robotNamespace>/</robotNamespace>
-        </plugin>
-    </gazebo>
+<?xml version="1.0"?>
+<robot xmlns:xacro="http://wiki.ros.org/xacro" name="$(arg robot_model)">
+   <!-- import main macro -->
+   <xacro:include filename="$(find ur_description)/urdf/inc/ur_macro.xacro"/>
+   <!-- parameters -->
+   <xacro:arg name="joint_limit_params" default=""/>
+   <xacro:arg name="kinematics_params" default=""/>
+   <xacro:arg name="physical_params" default=""/>
+   <xacro:arg name="visual_params" default=""/>
+   <!-- legal values:
+         - hardware_interface/PositionJointInterface
+         - hardware_interface/VelocityJointInterface
+         - hardware_interface/EffortJointInterface
+   -->
+   <xacro:arg name="transmission_hw_interface" default="hardware_interface/PositionJointInterface"/>
+   <xacro:arg name="safety_limits" default="false"/>
+   <xacro:arg name="safety_pos_margin" default="0.15"/>
+   <xacro:arg name="safety_k_position" default="20"/>
+   <!-- arm -->
+   <xacro:ur_robot
+     prefix=""
+     joint_limits_parameters_file="$(arg joint_limit_params)"
+     kinematics_parameters_file="$(arg kinematics_params)"
+     physical_parameters_file="$(arg physical_params)"
+     visual_parameters_file="$(arg visual_params)"
+     transmission_hw_interface="$(arg transmission_hw_interface)"
+     safety_limits="$(arg safety_limits)"
+     safety_pos_margin="$(arg safety_pos_margin)"
+     safety_k_position="$(arg safety_k_position)"/>
 </robot>

File: src/ur5_apla/urdf/ur5_apla_with_printhead.xacro (robot description, xacro)
@@ -1,6 +1,31 @@
 <?xml version="1.0"?>
 <robot xmlns:xacro="http://ros.org/wiki/xacro" name="ur5_apla_with_printhead">
-  <!-- ur5 -->
-  <xacro:include filename="$(find ur5_apla)/urdf/ur5_apla.xacro" />
+  <!-- import main macro -->
+  <xacro:include filename="$(find ur_description)/urdf/inc/ur_macro.xacro"/>
+  <!-- parameters -->
+  <xacro:arg name="joint_limit_params" default=""/>
+  <xacro:arg name="kinematics_params" default=""/>
+  <xacro:arg name="physical_params" default=""/>
+  <xacro:arg name="visual_params" default=""/>
+  <!-- legal values:
+        - hardware_interface/PositionJointInterface
+        - hardware_interface/VelocityJointInterface
+        - hardware_interface/EffortJointInterface
+  -->
+  <xacro:arg name="transmission_hw_interface" default="hardware_interface/PositionJointInterface"/>
+  <xacro:arg name="safety_limits" default="false"/>
+  <xacro:arg name="safety_pos_margin" default="0.15"/>
+  <xacro:arg name="safety_k_position" default="20"/>
+  <!-- arm -->
+  <xacro:ur_robot
+    prefix=""
+    joint_limits_parameters_file="$(arg joint_limit_params)"
+    kinematics_parameters_file="$(arg kinematics_params)"
+    physical_parameters_file="$(arg physical_params)"
+    visual_parameters_file="$(arg visual_params)"
+    transmission_hw_interface="$(arg transmission_hw_interface)"
+    safety_limits="$(arg safety_limits)"
+    safety_pos_margin="$(arg safety_pos_margin)"
+    safety_k_position="$(arg safety_k_position)"/>
   <!-- end-effector -->
   <xacro:include filename="$(find ur5_apla)/urdf/printhead.xacro" />
