Commit message: Refactor ur5_apla_with_printhead

File: src/ur5_apla/urdf/ur5_apla_with_printhead.xacro (robot description, xacro)
@@ -4,8 +4,8 @@
   <xacro:include filename="$(find ur_description)/urdf/inc/ur_macro.xacro"/>
   <!-- parameters -->
-  <xacro:arg name="joint_limit_params" default=""/>
-  <xacro:arg name="kinematics_params" default=""/>
-  <xacro:arg name="physical_params" default=""/>
-  <xacro:arg name="visual_params" default=""/>
+  <xacro:arg name="joint_limit_params" default="$(find ur5_apla)/config/joint_limits.yaml"/>
+  <xacro:arg name="kinematics_params" default="$(find ur5_apla)/config/ur5_apla_kinematics.yaml"/>
+  <xacro:arg name="physical_params" default="$(find ur5_apla)/config/physical_parameters.yaml"/>
+  <xacro:arg name="visual_params" default="$(find ur5_apla)/config/visual_parameters.yaml"/>
   <!-- legal values:
         - hardware_interface/PositionJointInterface
@@ -33,9 +33,9 @@
   <xacro:printhead prefix="" connected_to="tool0"/>
   <!-- define the ur5's position and orientation in the world coordinate system -->
-  <!--link name="world" />
+  <link name="world" />
   <joint name="world_joint" type="fixed">
     <parent link="world" />
     <child link="base_link" />
     <origin xyz="0.0 0.0 0.0" rpy="0.0 0.0 0.0" />
-  </joint>-->
+  </joint>
 </robot>

File: src/ur5_apla_moveit_config/config/gazebo_ur5_apla_with_printhead.urdf (robot description, URDF)
Before this commit: robot ur5_apla_with_printhead, 14 links, 13 joints
Links:
- link base_link_inertia: geometry collision mesh filename=package://ur_description/meshes/ur5/collision/base.stl; visual mesh filename=package://ur_description/meshes/ur5/visual/base.dae
- link forearm_link: geometry collision mesh filename=package://ur_description/meshes/ur5/collision/forearm.stl; visual mesh filename=package://ur_description/meshes/ur5/visual/forearm.dae
- link shoulder_link: geometry collision mesh filename=package://ur_description/meshes/ur5/collision/shoulder.stl; visual mesh filename=package://ur_description/meshes/ur5/visual/shoulder.dae
- link upper_arm_link: geometry collision mesh filename=package://ur_description/meshes/ur5/collision/upperarm.stl; visual mesh filename=package://ur_description/meshes/ur5/visual/upperarm.dae
- link wrist_1_link: geometry collision mesh filename=package://ur_description/meshes/ur5/collision/wrist1.stl; visual mesh filename=package://ur_description/meshes/ur5/visual/wrist1.dae
- link wrist_2_link: geometry collision mesh filename=package://ur_description/meshes/ur5/collision/wrist2.stl; visual mesh filename=package://ur_description/meshes/ur5/visual/wrist2.dae
- link wrist_3_link: geometry collision mesh filename=package://ur_description/meshes/ur5/collision/wrist3.stl; visual mesh filename=package://ur_description/meshes/ur5/visual/wrist3.dae
Joints:
- joint elbow_joint: origin xyz=-0.425 0 0 rpy=0 0 0 -> xyz=-0.4245346711001575 0 0 rpy=0.0002669342234943978 0.0002850281317621745 4.118411028599387e-05
- joint shoulder_lift_joint: origin xyz=0 0 0 rpy=1.570796327 0 0 -> xyz=0.0002106426285080585 0 0 rpy=1.570366839582577 0 4.170074070522014e-05
- joint shoulder_pan_joint: origin xyz=0 0 0.089159 rpy=0 0 0 -> xyz=0 0 0.08908222291512749 rpy=0 0 -4.019222839807838e-05
- joint wrist_1_joint: origin xyz=-0.39225 0 0.10915 rpy=0 0 0 -> xyz=-0.3915927671902 0.0005685293830529392 0.1107229976042442 rpy=3.136457998649264 3.139679965191397 3.141551453073033
- joint wrist_2_joint: origin xyz=0 -0.09465 -1.941303950897609e-11 rpy=1.570796327 0 0 -> xyz=-2.88761848246674e-05 -0.09474646855904763 9.819830366276481e-05 rpy=1.569759894830783 0 -0.000126022682877951
- joint wrist_3_joint: origin xyz=0 0.0823 -1.688001216681175e-11 rpy=1.570796326589793 3.141592653589793 3.141592653589793 -> xyz=0.0001192375579587692 0.08238710113518417 5.421843634149577e-05 rpy=1.571454420449939 3.141592653589793 3.141513767867271
