Commit message: Added the constraints of the workspace

File: src/ur5_apla/urdf/printhead.xacro (robot description, xacro)
@@ -15,5 +15,5 @@
         <geometry>
           <!-- The path to the visual meshes in the package. -->
-          <mesh filename="package://ur5_apla/meshes/printhead/visual/printhead.stl"/>
+          <mesh filename="package://ur5_apla/meshes/printhead/visual/printhead.dae"/>
         </geometry>
       </visual>
@@ -27,5 +27,5 @@
     <!-- TCP frame -->
     <joint name="${prefix}tcp_joint" type="fixed">
-      <origin xyz="0 0 0.116" rpy="0 0 0"/>
+      <origin xyz="0 0 0.19515" rpy="0 0 0"/>
       <parent link="${prefix}printhead"/>
       <child link="${prefix}tcp"/>

Commit message: Cleaning up

File: src/ur5_apla/urdf/printhead.xacro (robot description, xacro)
@@ -26,6 +26,7 @@
     </link>
     <!-- TCP frame -->
+    <!-- TCP is at 0.19515m according to .STL, after measuring appears to be 0.00286m further away -->
     <joint name="${prefix}tcp_joint" type="fixed">
-      <origin xyz="0 0 0.19515" rpy="0 0 0"/>
+      <origin xyz="0 0 0.19801" rpy="0 0 0"/>
       <parent link="${prefix}printhead"/>
       <child link="${prefix}tcp"/>

Commit message: Finished planar-positioning code

File: src/ur5_apla/urdf/printhead.xacro (robot description, xacro)
@@ -14,6 +14,6 @@
       <visual>
         <geometry>
-          <!-- The path to the visual meshes in the package. -->
-          <mesh filename="package://ur5_apla/meshes/printhead/visual/printhead.dae"/>
+          <!-- The path to the visual meshes in the package. This can be the dae variant -->
+          <mesh filename="package://ur5_apla/meshes/printhead/visual/printheadv2.stl"/>
         </geometry>
       </visual>
@@ -21,12 +21,13 @@
         <geometry>
           <!-- The path to the collision meshes in the package. -->
-          <mesh filename="package://ur5_apla/meshes/printhead/collision/printhead.stl"/>
+          <mesh filename="package://ur5_apla/meshes/printhead/collision/printheadv2.stl"/>
         </geometry>
       </collision>
     </link>
     <!-- TCP frame -->
-    <!-- TCP is at 0.19515m according to .STL, after measuring appears to be 0.00286m further away -->
+    <!-- TCP is at 0.19515m according to .STL, after measuring appears to be 0.00286m further away, old value with stool-head was 0.19801 -->
+    <!-- TCP is at 0.19515m according to initial .STL, after measuring appears to be 0.00162 further away, modified the .SLDASM so now TCP is at 0.19677-->
     <joint name="${prefix}tcp_joint" type="fixed">
-      <origin xyz="0 0 0.19801" rpy="0 0 0"/>
+      <origin xyz="0 0 0.19677" rpy="0 0 0"/>
       <parent link="${prefix}printhead"/>
       <child link="${prefix}tcp"/>

Commit message: details

File: src/ur5_apla/urdf/printhead.xacro (robot description, xacro)
@@ -15,5 +15,5 @@
         <geometry>
           <!-- The path to the visual meshes in the package. This can be the dae variant -->
-          <mesh filename="package://ur5_apla/meshes/printhead/visual/printheadv2.stl"/>
+          <mesh filename="package://ur5_apla/meshes/printhead/visual/printheadv2.dae"/>
         </geometry>
       </visual>

Commit message: Some final details

File: src/ur5_apla/urdf/printhead.xacro (robot description, xacro)
@@ -21,5 +21,5 @@
         <geometry>
           <!-- The path to the collision meshes in the package. -->
-          <mesh filename="package://ur5_apla/meshes/printhead/collision/printheadv2.stl"/>
+          <mesh filename="package://ur5_apla/meshes/printhead/collision/printheadv2.dae"/>
         </geometry>
       </collision>
